Commit message: improve pa scene and some bugs

File: baxter_description/urdf/baxter_base/baxter_base_ft2.urdf.xacro (robot description, xacro)
@@ -1046,5 +1046,5 @@
   </xacro:if>
   <xacro:unless value="$(arg left_ft_sensor)">
-    <joint name="right_hand" type="fixed">
+    <joint name="left_hand" type="fixed">
       <origin rpy="0 0 0" xyz="0 0 0.11355"/>
       <axis xyz="0 0 1"/>

File: baxter_description/urdf/baxter_full.urdf.xacro (robot description, xacro)
@@ -25,5 +25,5 @@
   <xacro:arg name="gazebo" value="$(arg gazebo)"/>
   <xacro:arg name="left_ft_sensor" value="$(arg left_ft_sensor)"/>
-  <xacro:arg name="right_ft_sensor" default="$(arg right_ft_sensor)"/>
+  <xacro:arg name="right_ft_sensor" value="$(arg right_ft_sensor)"/>
   </xacro:include>
   <!-- Baxter Pedestal -->

File: baxter_description/urdf/left_end_pa_effector.urdf.xacro (robot description, xacro)
@@ -5,5 +5,5 @@
   <xacro:arg name="l_finger_tip" default="paddle_tip"/>
   <xacro:arg name="l_finger_grasp" default="inner"/>
-  <xacro:arg name="left_camera_frame" default="fault"/>
+  <xacro:arg name="left_camera_frame" default="false"/>
   <xacro:include filename="$(find rethink_ee_description)/urdf/electric_gripper/rethink_electric_pa_gripper.xacro" />
   <xacro:rethink_electric_gripper side="left"

File: baxter_description/urdf/right_end_pa_effector.urdf.xacro (robot description, xacro)
@@ -5,5 +5,5 @@
   <xacro:arg name="r_finger_tip" default="paddle_tip"/>
   <xacro:arg name="r_finger_grasp" default="inner"/>
-  <xacro:arg name="right_camera_frame" default="fault"/>
+  <xacro:arg name="right_camera_frame" default="false"/>
   <xacro:include filename="$(find rethink_ee_description)/urdf/electric_gripper/rethink_electric_pa_gripper.xacro" />
   <xacro:rethink_electric_gripper side="right"

File: rethink_ee_description/urdf/electric_gripper/fingers/pa_finger.xacro (robot description, xacro)
@@ -6,5 +6,5 @@
     <link name="${gripper_side}_gripper_${finger_side}_finger">
       <visual>
-        <origin rpy="${-pi/2*reflect} ${pi/2+pi/2*reflect} 0" xyz="0 0 0"/>
+        <origin rpy="${-pi/2*reflect} ${pi/2+pi/2*reflect} 0" xyz="0 0 0.035"/>
         <geometry>
           <mesh filename="package://rethink_ee_description/meshes/electric_gripper/fingers/finger.dae"/>
@@ -12,5 +12,5 @@
       </visual>
       <collision>
-        <origin rpy="${-pi/2*reflect} ${pi/2+pi/2*reflect} 0" xyz="0 0 0"/>
+        <origin rpy="${-pi/2*reflect} ${pi/2+pi/2*reflect} 0" xyz="0 0 0.035"/>
         <geometry>
           <mesh filename="package://rethink_ee_description/meshes/electric_gripper/fingers/finger.stl"/>

File: rethink_ee_description/urdf/electric_gripper/fingers/pa_tip.xacro (robot description, xacro)
@@ -8,5 +8,5 @@
     <link name="${parent_link}_tip">
       <visual>
-        <origin rpy="0 0 0" xyz="0 ${-0.011*g_reflect} -0.005"/>
+        <origin rpy="0 0 0" xyz="0 ${-0.011*g_reflect} 0.03"/>
         <geometry>
           <box size="0.02 0.002 0.015"/>
@@ -14,5 +14,5 @@
       </visual>
       <collision>
-        <origin rpy="0 0 0" xyz="0 ${-0.011*g_reflect} -0.005"/>
+        <origin rpy="0 0 0" xyz="0 ${-0.011*g_reflect} 0.03"/>
         <geometry>
           <box size="0.02 0.002 0.015"/>

File: robots_description/robots/robot_system_config.urdf.xacro (robot description, xacro)
@@ -6,7 +6,21 @@
   <xacro:arg name="table" default="true"/>
   <xacro:arg name="asus_xtion" default="true"/>
+  <xacro:arg name="right_camera_frame" default="true"/>
+  <xacro:arg name="left_camera_frame" default="true"/>
+  <xacro:arg name="l_finger"       default="pa_finger"/>
+  <xacro:arg name="l_finger_slot"  default="6"/>
+  <xacro:arg name="l_finger_tip"   default="pa_tip"/>
+  <xacro:arg name="l_finger_grasp" default="inner"/>
+  <xacro:arg name="r_finger"       default="pa_finger"/>
+  <xacro:arg name="r_finger_slot"  default="6"/>
+  <xacro:arg name="r_finger_tip"   default="pa_tip"/>
+  <xacro:arg name="r_finger_grasp" default="inner"/>
+  <xacro:arg name="left_ft_sensor" default="false"/>
+  <xacro:arg name="right_ft_sensor" default="true"/>
   <!-- Baxter Base URDF -->
-  <xacro:include filename="$(find baxter_description)/urdf/baxter_base/baxter_base.urdf.xacro">
+  <xacro:include filename="$(find baxter_description)/urdf/baxter_base/baxter_base_ft2.urdf.xacro">
     <xacro:arg name="gazebo" value="${gazebo}"/>
+    <xacro:arg name="left_ft_sensor" value="$(arg left_ft_sensor)"/>
+    <xacro:arg name="right_ft_sensor" value="$(arg right_ft_sensor)"/>
   </xacro:include>
   <!-- Baxter Pedestal -->
@@ -17,7 +31,19 @@
   </xacro:if>
   <!-- Left End Effector -->
-  <xacro:include filename="$(find baxter_description)/urdf/left_end_pa_effector.urdf.xacro" />
-  <!-- Right End Effector -->
-  <xacro:include filename="$(find baxter_description)/urdf/right_end_pa_effector.urdf.xacro" />
+    <xacro:include filename="$(find baxter_description)/urdf/left_end_pa_effector.urdf.xacro" >
+      <xacro:arg name="left_camera_frame" default="$(left_camera_frame)"/>
+      <xacro:arg name="l_finger" default="$(l_finger)"/>
+      <xacro:arg name="l_finger_slot" default="$(l_finger_slot)"/>
+      <xacro:arg name="l_finger_tip" default="$(l_finger_tip)"/>
+      <xacro:arg name="l_finger_grasp" default="$(l_finger_grasp)"/>
+    </xacro:include>
+    <!-- Right End Effector -->
+    <xacro:include filename="$(find baxter_description)/urdf/right_end_pa_effector.urdf.xacro" >
+      <xacro:arg name="right_camera_frame" default="$(right_camera_frame)"/>
+      <xacro:arg name="r_finger" default="$(r_finger)"/>
+      <xacro:arg name="r_finger_slot" default="$(r_finger_slot)"/>
+      <xacro:arg name="r_finger_tip" default="$(r_finger_tip)"/>
+      <xacro:arg name="r_finger_grasp" default="$(r_finger_grasp)"/>
+    </xacro:include>
   <!-- Table -->
   <xacro:if value="$(arg table)">
